File: MCUTestBoard.kicad_sch (KiCad schematic)
At the start: 42 parts, among them J1 Conn_01x16, J2 Conn_01x16, J3 USB_B_Micro, J4 Conn_01x06, J5 Conn_01x16, J6 Conn_01x16, SW1 SW_Push, SW2 SW_SPDT, SW3 SW_SPDT, U1 QFP64-0.5-REV2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

Commit message: LED resistor 150R Add enclosure model add iBom
Parts:
- R2: value 130 -> 150
Changed lines of the file:
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@@
 			)
 		)
-		(property "Value" "130"
+		(property "Value" "150"
 			(at 91.44 176.53 90)
 			(effects
